Commit message: Kuka_arm

File: Simulation/New_arm/urdf/Cerebroarm.xacro (robot description, xacro)
@@ -1,103 +1,421 @@
-<?xml version="1.0" ?>
-<robot name="Cerebroarm" xmlns:xacro="http://www.ros.org/wiki/xacro">
-<xacro:property name="pi" value="3.1415926535897931"/>
-<xacro:property name="r1" value="0.06"/>
-<xacro:property name="l1" value="0.30"/>
-<xacro:property name="l2" value="0.40"/>
-<xacro:property name="m" value="1"/>
-<xacro:property name="a" value="0.50"/>
-<link name="world"/>
-<joint name="fixed" type="fixed">
-    <parent link="world"/>
-    <child  link="base_plate"/>
-</joint>
-<link name="base_plate">
-    <inertial>
-        <mass value="${m}"/>
-        <origin xyz="0.0 0.0 0.025" rpy="0.0 0.0 0.0"/>
-        <inertia ixx="0.020833" iyy="0.020833" izz="0.041667" iyz="0.0" ixz="0.0" ixy="0.0"/>
-    </inertial>
-    <visual>
-        <origin xyz="0 0 0.025" rpy="0.0 0.0 0.0"/>
-          <geometry>
-              <box size="${a} ${a} 0.05"/>
-          </geometry>
-    </visual>
-</link>
-<joint name="plate_basecyl" type="continuous">
-    <origin xyz="0.0 0.0 0.025" rpy="0.0 0.0 0.0"/>
-    <parent link="base_plate"/>
-    <child link="base_cylinder"/>
-    <axis xyz="0.0 1.0 0.0"/>
-</joint>
-<link name="base_cylinder">
-    <inertial>
-        <mass value="${m}"/>
-        <origin xyz="0 0 ${0.05+l1/2}" rpy="0.0 0.0 0.0"/>
-        <inertia ixx="${m/3.0*l1*l1}" iyy="${m/3.0*l1*l1}" izz="${m/2*r1*r1}" iyz="0.0" ixz="0.0" ixy="0.0" />
-    </inertial>
-    <visual>
-        <origin xyz="0 0 ${l1/2}" rpy="0.0 0.0 0.0"/>
-          <geometry>
-              <cylinder radius="${r1}" length="${l1}"/>
-          </geometry>
-    </visual>
-</link>
-<link name="base_cylinder1">
-    <inertial>
-        <mass value="${m}"/>
-        <origin xyz="0 0 ${0.05+1.5*l1}" rpy="0.0 0.0 0.0"/>
-        <inertia ixx="${m/3.0*l1*l1}" iyy="${m/3.0*l1*l1}" izz="${m/2*r1*r1}" iyz="0.0" ixz="0.0" ixy="0.0" />
-    </inertial>
-    <visual>
-        <origin xyz="0 0 ${l1/2}" rpy="0.0 0.0 0.0"/>
-          <geometry>
-              <cylinder radius="${r1}" length="${l1}"/>
-          </geometry>
-    </visual>
-</link>
-<joint name="basecyl_zaxis" type="continuous">
-    <origin xyz="0.0 0.0 ${l1}" rpy="0.0 0.0 0.0"/>
-    <parent link="base_cylinder"/>
-    <child link="base_cylinder1"/>
-    <axis xyz="0.0 0.0 1.0"/>
-</joint>
-<link name="base_cylinder2">
-    <inertial>
-        <mass value="${m}"/>
-        <origin xyz="0 0 ${0.05+2*l1+0.5*l2}" rpy="0.0 0.0 0.0"/>
-        <inertia ixx="${m/3.0*l1*l1}" iyy="${m/3.0*l1*l1}" izz="${m/2*r1*r1}" iyz="0.0" ixz="0.0" ixy="0.0" />
-    </inertial>
-    <visual>
-        <origin xyz="0 0 ${l2/2+l1/2-0.05}" rpy="0.0 0.0 0.0"/>
-          <geometry>
-              <cylinder radius="${r1}" length="${l1}"/>
-          </geometry>
-    </visual>
-</link>
-<joint name="basecyl_zaxis1" type="continuous">
-    <origin xyz="0.0 0.0 ${l1}" rpy="0.0 0.0 0.0"/>
-    <parent link="base_cylinder1"/>
-    <child link="base_cylinder2"/>
-    <axis xyz="1.0 0.0 0.0"/>
-</joint>
-<link name="gripper">
-    <inertial>
-        <mass value="${m}"/>
-        <origin xyz="0 0 ${0.05+2*l1+0.5*l2}" rpy="${pi/2} 0.0 0.0"/>
-        <inertia ixx="${m/3.0*l1*l1}" iyy="${m/3.0*l1*l1}" izz="${m/2*r1*r1}" iyz="0.0" ixz="0.0" ixy="0.0" />
-    </inertial>
-    <visual>
-        <origin xyz="0 0 ${l2/2+l1/2-0.05}" rpy="0.0 0.0 0.0"/>
-          <geometry>
-              <cylinder radius="${r1}" length="${l1}"/>
-          </geometry>
-    </visual>
-</link>
-<joint name="basecyl_zaxis2" type="continuous">
-    <origin xyz="0.0 0.0 ${l1}" rpy="0.0 0.0 0.0"/>
-    <parent link="base_cylinder2"/>
-    <child link="gripper"/>
-    <axis xyz="1.0 0.0 0.0"/>
-</joint>
+<?xml version="1.0"?>
+<robot name="cerebroarm" xmlns:xacro="http://www.ros.org/wiki/xacro">
+  <!--Define constants-->
+  <xacro:property name="pi" value="3.141592654"/>
+  <xacro:property name="deg" value="0.017453293"/><!--degrees to radians-->
+  <xacro:property name="mass0" value="150" />
+  <xacro:property name="mass1" value="138" />
+  <xacro:property name="mass2" value="95" />
+  <xacro:property name="mass3" value="71" />
+  <xacro:property name="mass4" value="17" />
+  <xacro:property name="mass5" value="7" />
+  <xacro:property name="mass6" value="0.5" />
+  <xacro:property name="gripper_mass" value="0.3" />
+  <xacro:property name="finger_mass" value="0.1" />
+  <xacro:property name="gripper_type" value="vacuum" />
+  <xacro:property name="vacuum_gripper_radius" value="0.1" />
+  <!--Import gazebo elements-->
+  <xacro:include filename="$(find arm)/src/URDF/kr210.gazebo.xacro" />
+  <!--Links-->
+  <link name="base_footprint"/>
+  <link name="base_link">
+    <inertial>
+      <origin xyz="0 0 0" rpy="0 0 0"/>
+      <mass value="${mass0}"/>
+      <inertia ixx="60" ixy="0" ixz="0" iyy="70" iyz="0" izz="100"/>
+    </inertial>
+    <visual>
+      <origin xyz="0 0 0" rpy="${-pi/2} 0 0"/>
+      <geometry>
+        <mesh filename="package://arm/meshes/kr210l150/visual/base_link.dae"/>
+      </geometry>
+      <material name="">
+        <color rgba="0.75294 0.75294 0.75294 1"/>
+      </material>
+    </visual>
+    <collision>
+      <origin xyz="0 0 0" rpy="${-pi/2} 0 0"/>
+      <geometry>
+        <mesh filename="package://arm/meshes/kr210l150/collision/base_link.stl"/>
+      </geometry>
+    </collision>
+  </link>
+  <link name="link_1">
+    <inertial>
+      <origin xyz="0 0 0.4" rpy="0 0 0"/>
+      <mass value="${mass1}"/>
+      <inertia ixx="30" ixy="0" ixz="0" iyy="50" iyz="0" izz="50"/>
+    </inertial>
+    <visual>
+      <origin xyz="0 0 0" rpy="0 0 0"/>
+      <geometry>
+        <mesh filename="package://arm/meshes/kr210l150/visual/link_1.dae"/>
+      </geometry>
+      <material name="">
+        <color rgba="0.75294 0.75294 0.75294 1"/>
+      </material>
+    </visual>
+    <collision>
+      <origin xyz="0 0 0" rpy="0 0 0"/>
+      <geometry>
+        <mesh filename="package://arm/meshes/kr210l150/collision/link_1.stl"/>
+      </geometry>
+    </collision>
+  </link>
+  <link name="link_2">
+    <inertial>
+      <origin xyz="0 0 0.44751" rpy="0 0 0"/>
+      <mass value="${mass2}"/>
+      <inertia ixx="40" ixy="0" ixz="0" iyy="40" iyz="0" izz="10"/>
+    </inertial>
+    <visual>
+      <origin xyz="0 0 0" rpy="${-pi/2} 0 0"/>
+      <geometry>
+        <mesh filename="package://arm/meshes/kr210l150/visual/link_2.dae"/>
+      </geometry>
+      <material name="">
+        <color rgba="0.75294 0.75294 0.75294 1"/>
+      </material>
+    </visual>
+    <collision>
+      <origin xyz="0 0 0" rpy="0 0 0"/>
+      <geometry>
+        <mesh filename="package://arm/meshes/kr210l150/collision/link_2.stl"/>
+      </geometry>
+    </collision>
+  </link>
+  <link name="link_3">
+    <inertial>
+      <origin xyz="0.18842 0.18344 -0.042799" rpy="0 0 0"/>
+      <mass value="${mass3}"/>
+      <inertia ixx="1" ixy="0" ixz="0" iyy="10" iyz="0" izz="10"/>
+    </inertial>
+    <visual>
+      <origin xyz="0 -0.184 0" rpy="${-pi/2} 0 0"/>
+      <geometry>
+        <mesh filename="package://arm/meshes/kr210l150/visual/link_3.dae"/>
+      </geometry>
+      <material name="">
+        <color rgba="0.75294 0.75294 0.75294 1"/>
+      </material>
+    </visual>
+    <collision>
+      <origin xyz="0 -0.184 0" rpy="0 0 0"/>
+      <geometry>
+        <mesh filename="package://arm/meshes/kr210l150/collision/link_3.stl"/>
+      </geometry>
+    </collision>
+  </link>
+  <link name="link_4">
+    <inertial>
+      <origin xyz="0.27146 -0.007326 0" rpy="0 0 0"/>
+      <mass value="${mass4}"/>
+      <inertia ixx="0.18" ixy="0" ixz="0" iyy="0.55" iyz="0" izz="0.64"/>
+    </inertial>
+    <visual>
+      <origin xyz="0 0 0" rpy="${-pi/2} 0 0"/>
+      <geometry>
+        <mesh filename="package://arm/meshes/kr210l150/visual/link_4.dae"/>
+      </geometry>
+      <material name="">
+        <color rgba="0.75294 0.75294 0.75294 1"/>
+      </material>
+    </visual>
+    <collision>
+      <origin xyz="0 0 0" rpy="0 0 0"/>
+      <geometry>
+        <mesh filename="package://arm/meshes/kr210l150/collision/link_4.stl"/>
+      </geometry>
+    </collision>
+  </link>
+  <link name="link_5">
+    <inertial>
+      <origin xyz="0 0 0" rpy="0 0 0"/>
+      <mass value="${mass5}"/>
+      <inertia ixx="0.04" ixy="0" ixz="0" iyy="0.068" iyz="0" izz="0.068"/>
+    </inertial>
+    <visual>
+      <origin xyz="0 0 0" rpy="${-pi/2} 0 0"/>
+      <geometry>
+        <mesh filename="package://arm/meshes/kr210l150/visual/link_5.dae"/>
+      </geometry>
+      <material name="">
+        <color rgba="0.75294 0.75294 0.75294 1"/>
+      </material>
+    </visual>
+    <collision>
+      <origin xyz="0 0 0" rpy="0 0 0"/>
+      <geometry>
+        <mesh filename="package://arm/meshes/kr210l150/collision/link_5.stl"/>
+      </geometry>
+    </collision>
+  </link>
+  <link name="link_6">
+    <inertial>
+      <origin xyz="0 0 0" rpy="0 0 0"/>
+      <mass value="${mass6}"/>
+      <inertia ixx="0.004" ixy="0" ixz="0" iyy="0.003" iyz="0" izz="0.003"/>
+    </inertial>
+    <visual>
+      <origin xyz="0 0 0" rpy="0 0 0"/>
+      <geometry>
+        <mesh filename="package://arm/meshes/kr210l150/visual/link_6.dae"/>
+      </geometry>
+      <material name="">
+        <color rgba="0.75294 0.75294 0.75294 1"/>
+      </material>
+    </visual>
+    <collision>
+      <origin xyz="0 0 0" rpy="0 0 0"/>
+      <geometry>
+        <mesh filename="package://arm/meshes/kr210l150/collision/link_6.stl"/>
+      </geometry>
+    </collision>
+  </link>
+  <!--Gripper links-->
+  <!--Vacuum gripper-->
+  <xacro:if value="${gripper_type == 'vacuum'}">
+  <link name="gripper_link">
+    <inertial>
+      <origin xyz="0 0 0" rpy="0 0 0"/>
+      <mass value="${gripper_mass}"/>
+      <inertia ixx="0.005" ixy="0" ixz="0" iyy="0.00" iyz="0" izz="0.00"/>
+    </inertial>
+    <visual>
+      <origin xyz="0 0 0" rpy="0 0 0"/>
+      <geometry>
+        <sphere radius="${vacuum_gripper_radius}"/>
+      </geometry>
+    </visual>
+    <collision>
+      <origin xyz="0 0 0" rpy="0 0 0"/>
+      <geometry>
+        <sphere radius="${vacuum_gripper_radius}"/>
+      </geometry>
+    </collision>
+  </link>
+  <joint name="gripper_joint" type="fixed">
+    <parent link="link_6"/>
+    <child link="gripper_link"/>
+    <origin xyz="0.0375 0 0" rpy="0 0 0"/>
+  </joint>
+  </xacro:if>
+  <!--Two-finger gripper-->
+  <xacro:if value="${gripper_type == 'two_finger'}">
+  <link name="gripper_link">
+    <inertial>
+      <origin xyz="0 0 0" rpy="0 0 0"/>
+      <mass value="${gripper_mass}"/>
+      <inertia ixx="0.0001" ixy="0" ixz="0" iyy="0.0002" iyz="0" izz="0.0001"/>
+    </inertial>
+    <visual>
+      <origin xyz="0 0 0" rpy="0 0 0"/>
+      <geometry>
+        <mesh filename="package://arm/meshes/gripper/gripper_base.dae"/>
+      </geometry>
+    </visual>
+    <collision>
+      <origin xyz="0 0 0" rpy="0 0 0"/>
+      <geometry>
+        <mesh filename="package://arm/meshes/gripper/gripper_base.dae"/>
+      </geometry>
+    </collision>
+  </link>
+  <link name="right_gripper_finger_link">
+    <inertial>
+      <origin xyz="0 0 0" rpy="0 0 0"/>
+      <mass value="${finger_mass}"/>
+      <inertia ixx="0.002" ixy="0" ixz="0" iyy="0.0002" iyz="0" izz="0.0002"/>
+    </inertial>
+    <visual>
+      <origin xyz="0 0 0" rpy="0 0 0"/>
+      <geometry>
+        <mesh filename="package://arm/meshes/gripper/finger_right.dae"/>
+      </geometry>
+    </visual>
+    <collision>
+      <origin xyz="0 0 0" rpy="0 0 0"/>
+      <geometry>
+        <mesh filename="package://arm/meshes/gripper/finger_right_collision.dae"/>
+      </geometry>
+    </collision>
+  </link>
+  <link name="left_gripper_finger_link">
+    <inertial>
+      <origin xyz="0 0 0" rpy="0 0 0"/>
+      <mass value="${finger_mass}"/>
+      <inertia ixx="0.002" ixy="0" ixz="0" iyy="0.0002" iyz="0" izz="0.0002"/>
+    </inertial>
+    <visual>
+      <origin xyz="0 0 0" rpy="0 0 0"/>
+      <geometry>
+        <mesh filename="package://arm/meshes/gripper/finger_left.dae"/>
+      </geometry>
+    </visual>
+    <collision>
+      <origin xyz="0 0 0" rpy="0 0 0"/>
+      <geometry>
+        <mesh filename="package://arm/meshes/gripper/finger_left_collision.dae"/>
+      </geometry>
+    </collision>
+  </link>
+  <joint name="right_gripper_finger_joint" type="prismatic">
+    <origin rpy="0 0 0" xyz="0.15 -0.0725 0" />
+    <parent link="gripper_link" />
+    <child link="right_gripper_finger_link" />
+    <axis xyz="0 1 0" />
+    <limit effort="100" lower="-0.01" upper="0.06" velocity="0.05" />
+    <dynamics damping="0.7" />
+  </joint>
+  <joint name="left_gripper_finger_joint" type="prismatic">
+    <origin rpy="0 0 0" xyz="0.15 0.0725 0" />
+    <parent link="gripper_link" />
+    <child link="left_gripper_finger_link" />
+    <axis xyz="0 -1 0" />
+    <limit effort="100" lower="-0.01" upper="0.06" velocity="0.05" />
+    <dynamics damping="0.7" />
+  </joint>
+  <joint name="gripper_joint" type="fixed">
+    <parent link="link_6"/>
+    <child link="gripper_link"/>
+    <origin xyz="0.11 0 0" rpy="0 0 0"/><!--0.087-->
+    <axis xyz="0 1 0" />
+  </joint>
+  <transmission name="tran7">
+    <type>transmission_interface/SimpleTransmission</type>
+    <joint name="left_gripper_finger_joint">
+      <hardwareInterface>hardware_interface/EffortJointInterface</hardwareInterface>
+    </joint>
+    <actuator name="motor7">
+      <hardwareInterface>hardware_interface/EffortJointInterface</hardwareInterface>
+      <mechanicalReduction>1</mechanicalReduction>
+    </actuator>
+  </transmission>
+  <transmission name="tran8">
+    <type>transmission_interface/SimpleTransmission</type>
+    <joint name="right_gripper_finger_joint">
+      <hardwareInterface>hardware_interface/EffortJointInterface</hardwareInterface>
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